Commit message: mrsim rover: rear camera plus SDF spawn so both cameras publish
Add a rear-facing camera (camera_back_mount/link/optical, back_cam
sensor, camera_back_ros plugin on /camera_back/*) pitched down like
the front one, giving the fishtail row-change work a behind view.

Two spawn bugs fixed, both verified needed:
- distinct plugin names: two libgazebo_ros_camera plugins sharing one
  name race for the ROS node, the second never publishes.
- spawn from converted rover.sdf (-file) instead of the URDF topic:
  Gazebo 11 live URDF parsing drops the second camera sensor (only
  front_cam on gz transport), the SDF keeps both.

setup.py installs rover.sdf; farm.launch.py and farm_probe.launch.py
spawn -file rover.sdf while robot_state_publisher keeps the URDF.
Regenerate after URDF edits:
  gz sdf -p src/mrsim/urdf/rover.urdf > src/mrsim/urdf/rover.sdf

Verified on farm_maize: both gz sensors plus /camera/* and
/camera_back/* ROS topics; grabbed frames show crop rows ahead and
behind.

File: LinReg/MultiROI/tests/sim_ros2/src/mrsim/urdf/rover.urdf (robot description, URDF)
Before this commit: robot mrsim_rover, 10 links, 9 joints
Links:
- added link camera_back_link
- added link camera_back_mount; visual box size=0.10 0.08 0.06
- added link camera_back_optical
Joints:
- added joint camera_back_link_joint: type fixed, parent camera_back_mount, child camera_back_link, origin xyz=-0.06 0 0.05 rpy=0 0.42 3.14159265
- added joint camera_back_mount_joint: type fixed, parent base_link, child camera_back_mount, origin xyz=-0.22 0 1.15 rpy=0 0 0
- added joint camera_back_optical_joint: type fixed, parent camera_back_link, child camera_back_optical, origin xyz=0 0 0 rpy=-1.57079632679 0 -1.57079632679

Commit message: mrsim rover: ToF ranger hardware (side and angled front modules)
Add four ray-sensor modules to rover.urdf, all publishing
sensor_msgs/Range through libgazebo_ros_ray_sensor.so (5-ray fan,
infrared): tof_left/tof_right yawed +-90 deg at the chassis flanks,
tof_front_left/tof_front_right at the nose yawed +-35 deg outward so
head-on drift at bends is seen ahead. Every module has a small orange
housing box plus a dark stalk mast, all visual-only, so the sensors are
visible in the GUI without adding collision geometry.

The modules sit at z=0.30 on their stalks (beams at 0.46 m world):
high enough to clear the wheels and chassis top, low enough to stay
inside the 0..0.6 m plant stem band. An earlier revision at deck height
self-blinded all four channels at a constant 0.146 m on wheel and
chassis grazes; the raised mounts read clean inf in an empty world.
rover.sdf regenerated with gz sdf -p (the sim spawns the SDF, not the
URDF, because Gazebo 11 live URDF parsing drops the rear camera).

File: LinReg/MultiROI/tests/sim_ros2/src/mrsim/urdf/rover.urdf (robot description, URDF)
Before this commit: robot mrsim_rover, 13 links, 12 joints
Links:
- added link tof_fl_link; visual box size=0.03 0.03 0.20; visual box size=0.07 0.05 0.04
- added link tof_fr_link; visual box size=0.03 0.03 0.20; visual box size=0.07 0.05 0.04
- added link tof_left_link; visual box size=0.03 0.03 0.20; visual box size=0.07 0.05 0.04
- added link tof_right_link; visual box size=0.03 0.03 0.20; visual box size=0.07 0.05 0.04
Joints:
- added joint tof_fl_joint: type fixed, parent base_link, child tof_fl_link, origin xyz=0.24 0.18 0.30 rpy=0 0 0.6108652382
- added joint tof_fr_joint: type fixed, parent base_link, child tof_fr_link, origin xyz=0.24 -0.18 0.30 rpy=0 0 -0.6108652382
- added joint tof_left_joint: type fixed, parent base_link, child tof_left_link, origin xyz=0.10 0.24 0.30 rpy=0 0 1.57079632679
- added joint tof_right_joint: type fixed, parent base_link, child tof_right_link, origin xyz=0.10 -0.24 0.30 rpy=0 0 -1.57079632679
